File: waterputv4Schematics/waterputv4Schematics.kicad_sch (KiCad schematic)
At the start: 4 parts, among them J1 QDY30A, J2 Barrel_Jack, U1 ESP32-DEVKITC, U2 MAX485_MODULE_5V_LOGIC_TLL_TO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

Commit message: Final code
Parts:
- J1: footprint (none) -> Connector_JST:JST_XH_B4B-XH-AM_1x04_P2.50mm_Vertical
Connections:
- net GND2: now also U1.14 (GND1), U1.32 (GND2)
- no-connect marks 0 -> 31
Other:
- title: (none) -> Waterput V4
- moved on the sheet: J2
Changed lines of the file:
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@@
 (kicad_sch (version 20211123) (generator eeschema)
   (paper "A4")
+  (title_block
+    (title "Waterput V4")
+    (date "2025-09-15")
+    (rev "V1")
+  )
   (junction (at 148.59 88.9) (diameter 0) (color 0 0 0 0)
+  )
+  (no_connect (at 111.76 76.2))
+  (no_connect (at 111.76 78.74))
+  (no_connect (at 111.76 83.82))
+  (no_connect (at 111.76 81.28))
+  (no_connect (at 111.76 71.12))
+  (no_connect (at 111.76 73.66))
+  (no_connect (at 111.76 55.88))
+  (no_connect (at 111.76 58.42))
+  (no_connect (at 111.76 66.04))
+  (no_connect (at 111.76 86.36))
+  (no_connect (at 71.12 68.58))
+  (no_connect (at 71.12 66.04))
+  (no_connect (at 71.12 63.5))
+  (no_connect (at 71.12 60.96))
+  (no_connect (at 71.12 58.42))
+  (no_connect (at 111.76 96.52))
+  (no_connect (at 111.76 99.06))
+  (no_connect (at 71.12 96.52))
+  (no_connect (at 71.12 55.88))
+  (no_connect (at 71.12 53.34))
+  (no_connect (at 111.76 91.44))
+  (no_connect (at 111.76 93.98))
+  (no_connect (at 71.12 93.98))
+  (no_connect (at 71.12 91.44))
+  (no_connect (at 71.12 88.9))
+  (no_connect (at 71.12 83.82))
+  (no_connect (at 71.12 81.28))
+  (no_connect (at 71.12 78.74))
+  (no_connect (at 71.12 76.2))
+  (no_connect (at 71.12 73.66))
+  (no_connect (at 71.12 71.12))
+  (wire (pts (xy 69.85 86.36) (xy 71.12 86.36))
+    (stroke (width 0) (type default) (color 0 0 0 0))
   )
   (wire (pts (xy 180.34 87.63) (xy 179.07 87.63))
@@
     (pin "1")
   )
+  (symbol (lib_id "power:GND2") (at 69.85 86.36 270) (unit 1)
+    (in_bom yes) (on_board yes)
+    (property "Reference" "#PWR?" (id 0) (at 63.5 86.36 0)
+      (effects (font (size 1.27 1.27)) hide)
+    )
+    (property "Value" "GND2" (id 1) (at 60.96 86.36 90)
+      (effects (font (size 1.27 1.27)) (justify left))
+    )
+    (property "Footprint" "" (id 2) (at 69.85 86.36 0)
+      (effects (font (size 1.27 1.27)) hide)
+    )
+    (property "Datasheet" "" (id 3) (at 69.85 86.36 0)
+      (effects (font (size 1.27 1.27)) hide)
+    )
+    (pin "1")
+  )
   (symbol (lib_id "power:+5V") (at 179.07 80.01 270) (unit 1)
     (in_bom yes) (on_board yes) (fields_autoplaced)
@@
     (pin "1")
   )
-  (symbol (lib_id "power:+24V") (at 80.01 138.43 270) (unit 1)
-    (in_bom yes) (on_board yes) (fields_autoplaced)
-    (property "Reference" "#PWR0102" (id 0) (at 76.2 138.43 0)
-      (effects (font (size 1.27 1.27)) hide)
-    )
-    (property "Value" "+24V" (id 1) (at 83.82 138.4299 90)
-      (effects (font (size 1.27 1.27)) (justify left))
-    )
-    (property "Footprint" "" (id 2) (at 80.01 138.43 0)
-      (effects (font (size 1.27 1.27)) hide)
-    )
-    (property "Datasheet" "" (id 3) (at 80.01 138.43 0)
+  (symbol (lib_id "power:+24V") (at 250.19 82.55 270) (unit 1)
+    (in_bom yes) (on_board yes) (fields_autoplaced)
+    (property "Reference" "#PWR0102" (id 0) (at 246.38 82.55 0)
+      (effects (font (size 1.27 1.27)) hide)
+    )
+    (property "Value" "+24V" (id 1) (at 254 82.5499 90)
+      (effects (font (size 1.27 1.27)) (justify left))
+    )
+    (property "Footprint" "" (id 2) (at 250.19 82.55 0)
+      (effects (font (size 1.27 1.27)) hide)
+    )
+    (property "Datasheet" "" (id 3) (at 250.19 82.55 0)
       (effects (font (size 1.27 1.27)) hide)
     )
@@
     (pin "1")
   )
-  (symbol (lib_id "Connector:Barrel_Jack") (at 72.39 140.97 0) (unit 1)
-    (in_bom yes) (on_board yes) (fields_autoplaced)
-    (property "Reference" "J2" (id 0) (at 72.39 132.08 0))
-    (property "Value" "Barrel_Jack" (id 1) (at 72.39 134.62 0))
-    (property "Footprint" "Connector_BarrelJack:BarrelJack_Horizontal" (id 2) (at 73.66 141.986 0)
-      (effects (font (size 1.27 1.27)) hide)
-    )
-    (property "Datasheet" "~" (id 3) (at 73.66 141.986 0)
+  (symbol (lib_id "Connector:Barrel_Jack") (at 242.57 85.09 0) (unit 1)
+    (in_bom yes) (on_board yes) (fields_autoplaced)
+    (property "Reference" "J2" (id 0) (at 242.57 76.2 0))
+    (property "Value" "Barrel_Jack" (id 1) (at 242.57 78.74 0))
+    (property "Footprint" "Connector_BarrelJack:BarrelJack_Horizontal" (id 2) (at 243.84 86.106 0)
+      (effects (font (size 1.27 1.27)) hide)
+    )
+    (property "Datasheet" "~" (id 3) (at 243.84 86.106 0)
       (effects (font (size 1.27 1.27)) hide)
     )
     (pin "1")
     (pin "2")
+  )
+  (symbol (lib_id "power:GND2") (at 111.76 68.58 90) (unit 1)
+    (in_bom yes) (on_board yes) (fields_autoplaced)
+    (property "Reference" "#PWR?" (id 0) (at 118.11 68.58 0)
+      (effects (font (size 1.27 1.27)) hide)
+    )
+    (property "Value" "GND2" (id 1) (at 115.57 68.5799 90)
+      (effects (font (size 1.27 1.27)) (justify right))
+    )
+    (property "Footprint" "" (id 2) (at 111.76 68.58 0)
+      (effects (font (size 1.27 1.27)) hide)
+    )
+    (property "Datasheet" "" (id 3) (at 111.76 68.58 0)
+      (effects (font (size 1.27 1.27)) hide)
+    )
+    (pin "1")
   )
   (symbol (lib_id "power:GND1") (at 208.28 81.28 270) (unit 1)
@@
     (pin "1")
   )
-  (symbol (lib_id "power:GND1") (at 80.01 143.51 90) (unit 1)
-    (in_bom yes) (on_board yes) (fields_autoplaced)
-    (property "Reference" "#PWR0101" (id 0) (at 86.36 143.51 0)
-      (effects (font (size 1.27 1.27)) hide)
-    )
-    (property "Value" "GND1" (id 1) (at 83.82 143.5099 90)
+  (symbol (lib_id "power:GND1") (at 250.19 87.63 90) (unit 1)
+    (in_bom yes) (on_board yes) (fields_autoplaced)
+    (property "Reference" "#PWR0101" (id 0) (at 256.54 87.63 0)
+      (effects (font (size 1.27 1.27)) hide)
+    )
+    (property "Value" "GND1" (id 1) (at 254 87.6299 90)
       (effects (font (size 1.27 1.27)) (justify right))
     )
-    (property "Footprint" "" (id 2) (at 80.01 143.51 0)
-      (effects (font (size 1.27 1.27)) hide)
-    )
-    (property "Datasheet" "" (id 3) (at 80.01 143.51 0)
+    (property "Footprint" "" (id 2) (at 250.19 87.63 0)
+      (effects (font (size 1.27 1.27)) hide)
+    )
+    (property "Datasheet" "" (id 3) (at 250.19 87.63 0)
       (effects (font (size 1.27 1.27)) hide)
     )
@@
       (effects (font (size 1.27 1.27)) (justify left))
     )
-    (property "Footprint" "" (id 2) (at 213.36 83.82 0)
+    (property "Footprint" "Connector_JST:JST_XH_B4B-XH-AM_1x04_P2.50mm_Vertical" (id 2) (at 213.36 83.82 0)
       (effects (font (size 1.27 1.27)) hide)
     )
@@
       (reference "#PWR0108") (unit 1) (value "+5V") (footprint "")
     )
+    (path "/3d8ebf45-8705-4bcd-ab6d-fa107742e92e"
+      (reference "#PWR?") (unit 1) (value "GND2") (footprint "")
+    )
+    (path "/b92c6c4d-d632-492b-beae-1acdae4d089f"
+      (reference "#PWR?") (unit 1) (value "GND2") (footprint "")
+    )
     (path "/f14310e7-8d76-4aab-a4e5-69177ce4ba82"
